File: power.kicad_sch (KiCad schematic)
At the start: 8 parts, among them U1 LM2596S-5, U2 TLV1117-33

Commit message: Added some details
Other:
- note added: "The capacitor essentially takes in all the voltage when the power is on and when the switch is off it slowly discharges it, preventing the sudden up down of PWM."
- note added: "The inductor basically is a capacitor but it stores electric energy in a magnetic field. Inductance is the tendency to resist current changes. Steady current means the inductor is just a wire, when the current changes the inductor pushes back. This is basically used to smooth out the CURRENT coming out of the buck converter."
- note added: "This is a buck converter. It steps down voltage. By switching the voltage on and off over and over again, the average voltage outputted decreases."
- note added: "This is the power management schematic which takes 24V from the LiPo Battery and steps it down to 3V3 voltage for the STM32"
- note added: "This series of capacitors, inductors and diodes is to make the square wave voltage created by the buck converter into something more continuous for the circuits to use"
- moved on the sheet: C1, C2, C3, C4, D1, L1, U1, U2
